Commit message: Validate colour channels, and document the ROS packages some modules need

File: examples/robot_arm/robot.urdf (robot description, URDF)
Before this commit: robot example_arm, 5 links, 4 joints
Joints:
- joint finger_left_joint: origin xyz=0.3 0 0 -> xyz=0.3 0.0075 0
- joint finger_right_joint: origin xyz=0.3 0 0 -> xyz=0.3 -0.0075 0
